File: backlight-driver-niko.kicad_sch (KiCad schematic)
At the start: 14 parts

Commit message: Nikolite reviewed, silkscreen improved, added fuse, fixed a few small things wrt layout/sch
Parts:
- added F1: BL_Fuse, Fuse:Fuse_0805_2012Metric, symbol Device:Fuse_Small
- added R8, R9: 20K, Resistor_SMD:R_0402_1005Metric, symbol Device:R
- C3: value 22uF -> 1uF
- R1: value R -> 430K
- R2, R4, R5, R6: value R -> 20K
- R3: value R -> 560K
- R7: value 4.7K -> 5.1K
Connections:
- net +3V3: now also R9.2
- net GND: now also R8.1
- net L_FAULT: now also J1.4 (Enable), R9.1
- net L_PWM: now also J1.3 (PWM), R8.2
- net VAD: now also F1.1; no longer J1.1 (VAD)
- new net: F1.2, J1.1 (VAD)
- no-connect marks 6 -> 5
